File: PCBs/crosses-wired-thumb-cluster.kicad_pcb (KiCad board)
At the start: 2 copper layers, 126.8 x 111 mm, 44 parts, among them J1 Conn_01x06_Socket, J2 Conn_01x06_Socket, J4 Conn_01x14_Pin, J5 Conn_01x14_Pin, P1 TYPE-C-31-M-12 USB, P2 TYPE-C-31-M-12 USB, U1 supermini nrf / nice nano v2, U2 supermini nrf / nice nano v2

Commit message: Fixup old release
Parts:
- removed G***: LOGO, art-warning:gggw-logo
- removed the MB5 at (129.5, 162.2)
- removed the REF** at (195.0, 187.0)
- added J3: Conn_01x02_Socket, Connector_JST:JST_PH_S2B-PH-SM4-TB_1x02-1MP_P2.00mm_Horizontal, B.Cu at (200.3, 156.1)
- added J6: Conn_01x02_Socket, Connector_JST:JST_PH_S2B-PH-SM4-TB_1x02-1MP_P2.00mm_Horizontal, B.Cu at (112.0, 127.3)
- added JP1: SolderJumper_2_Open, Jumper:SolderJumper-2_P1.3mm_Open_RoundedPad1.0x1.5mm, B.Cu at (208.9, 158.4)
- added JP2: SolderJumper_2_Open, Jumper:SolderJumper-2_P1.3mm_Open_RoundedPad1.0x1.5mm, B.Cu at (114.7, 119.9)
- added REF**: KiCad-Logo2_5mm_SilkScreen, Symbol:KiCad-Logo2_5mm_SilkScreen, F.Cu at (176.1, 195.8)
- J1, J2: value Conn_01x06_Socket -> SM06B-SRSS-TB(LF)(SN); footprint PCM_marbastlib-xp-various:SM06B-SRSS-TB(LF)(SN) -> Connector_JST:JST_SH_SM06B-SRSS-TB_1x06-1MP_P1.00mm_Horizontal
- J4, J5: footprint Connector_FFC-FPC:Hirose_FH12-14S-0.5SH_1x14-1MP_P0.50mm_Horizontal -> PCM_marbastlib-various:XUNPU_FPC-05F-14PH20_1x14-1MP_P0.5mm_Horizontal
- moved J4 0.78 mm to (172.0, 153.0)
- moved J5 0.78 mm to (115.3, 157.0)
Connections:
- J1 pad 1: L-VCC -> GND
- J1 pad 2: L-SCK -> L-CS
- J1 pad 3: L-MOSI -> L-MISO
- J1 pad 4: L-MISO -> L-MOSI
- J1 pad 5: L-CS -> L-SCK
- J1 pad 6: GND -> L-VCC
- J2 pad 1: R-VCC -> GND
- J2 pad 2: R-SCK -> R-CS
- J2 pad 3: R-MOSI -> R-MISO
- J2 pad 4: R-MISO -> R-MOSI
- J2 pad 5: R-CS -> R-SCK
- J2 pad 6: GND -> R-VCC
- P1 pad A4: L-VCC -> VBATTL
- P1 pad A9: L-VCC -> VBATTL
- P1 pad B4: L-VCC -> VBATTL
- P1 pad B9: L-VCC -> VBATTL
- P2 pad A4: R-VCC -> VBATTR
- P2 pad A9: R-VCC -> VBATTR
- P2 pad B4: R-VCC -> VBATTR
- P2 pad B9: R-VCC -> VBATTR
- U1 pad 13: L-COLP -> VBATTL
- U1 pad 2: unconnected-(U1-D2-RX-Pad2) -> L-COLP
- U2 pad 13: R-COLP -> VBATTR
- U2 pad 2: unconnected-(U2-D2-RX-Pad2) -> R-COLP
Routing:
- net VBATTL: track 0.00 -> 22.4 mm
- net VBATTR: track 0.00 -> 17.7 mm
- net R-VCC: track 69.7 -> 54.7 mm
- net Net-(J3-Pin_2): track 0.00 -> 14.5 mm
- net L-VCC: track 75.9 -> 61.5 mm
- net Net-(J6-Pin_2): track 0.00 -> 13.9 mm
- net R-COLP: track 55.4 -> 52.1 mm
- net L-MISO: track 59.7 -> 60.6 mm
- net L-ROW3: track 49.0 -> 49.7 mm
- net L-COLP: track 49.0 -> 48.4 mm
- net GND: vias 54 -> 59
Other:
- outline, holes or cut-outs redrawn
- board text added: "CROSSES REV12"
- board text added: "FOR USE WITH REV2 FIRMWARE"
- board text removed: "CROSSES REV10"
- board text removed: "YOU ARE AWESOME"

Commit message: Changing license, adding wireless Gerbers, PCBs, etc
Parts:
- removed J3, J6: Conn_01x02_Socket, Connector_JST:JST_PH_S2B-PH-SM4-TB_1x02-1MP_P2.00mm_Horizontal
- removed JP1, JP2: SolderJumper_2_Open, Jumper:SolderJumper-2_P1.3mm_Open_RoundedPad1.0x1.5mm
- removed the REF** at (176.1, 195.8)
- added G***: LOGO, art-warning:gggw-logo, F.Cu at (174.9, 126.7)
- added MB5: 5.5mm, PCM_marbastlib-various:mousebites_5p5mm_easysnap, F.Cu at (129.5, 162.2)
- added REF**: KiCad-Logo2_12mm_SilkScreen, Symbol:KiCad-Logo2_12mm_SilkScreen, F.Cu at (195.0, 187.0)
- J1, J2: value SM06B-SRSS-TB(LF)(SN) -> Conn_01x06_Socket; footprint Connector_JST:JST_SH_SM06B-SRSS-TB_1x06-1MP_P1.00mm_Horizontal -> PCM_marbastlib-xp-various:SM06B-SRSS-TB(LF)(SN)
- J4, J5: footprint PCM_marbastlib-various:XUNPU_FPC-05F-14PH20_1x14-1MP_P0.5mm_Horizontal -> Connector_FFC-FPC:Hirose_FH12-14S-0.5SH_1x14-1MP_P0.50mm_Horizontal
- moved J4 0.78 mm to (172.0, 152.2)
- moved J5 0.78 mm to (116.0, 157.0)
Connections:
- J1 pad 1: GND -> L-VCC
- J1 pad 2: L-CS -> L-SCK
- J1 pad 3: L-MISO -> L-MOSI
- J1 pad 4: L-MOSI -> L-MISO
- J1 pad 5: L-SCK -> L-CS
- J1 pad 6: L-VCC -> GND
- J2 pad 1: GND -> R-VCC
- J2 pad 2: R-CS -> R-SCK
- J2 pad 3: R-MISO -> R-MOSI
- J2 pad 4: R-MOSI -> R-MISO
- J2 pad 5: R-SCK -> R-CS
- J2 pad 6: R-VCC -> GND
- P1 pad A4: VBATTL -> L-VCC
- P1 pad A9: VBATTL -> L-VCC
- P1 pad B4: VBATTL -> L-VCC
- P1 pad B9: VBATTL -> L-VCC
- P2 pad A4: VBATTR -> R-VCC
- P2 pad A9: VBATTR -> R-VCC
- P2 pad B4: VBATTR -> R-VCC
- P2 pad B9: VBATTR -> R-VCC
- U1 pad 13: VBATTL -> L-COLP
- U1 pad 2: L-COLP -> unconnected-(U1-D2-RX-Pad2)
- U2 pad 13: VBATTR -> R-COLP
- U2 pad 2: R-COLP -> unconnected-(U2-D2-RX-Pad2)
Routing:
- net VBATTL: track 22.4 -> 0.00 mm
- net VBATTR: track 17.7 -> 0.00 mm
- net R-VCC: track 54.7 -> 69.7 mm
- net Net-(J3-Pin_2): track 14.5 -> 0.00 mm
- net L-VCC: track 61.5 -> 75.9 mm
- net Net-(J6-Pin_2): track 13.9 -> 0.00 mm
- net R-COLP: track 52.1 -> 55.4 mm
- net L-MISO: track 60.6 -> 59.7 mm
- net L-ROW3: track 49.7 -> 49.0 mm
- net L-COLP: track 48.4 -> 49.0 mm
- net GND: vias 59 -> 54
Other:
- outline, holes or cut-outs redrawn
- board text added: "CROSSES REV10"
- board text added: "YOU ARE AWESOME"
- board text removed: "CROSSES REV12"
- board text removed: "FOR USE WITH REV2 FIRMWARE"
